Commit message: tiago with pal gripper description

File: robots/tiago.urdf.xacro (robot description, xacro)
@@ -17,4 +17,6 @@
     <xacro:arg name="multiple" default="false"/>
     <xacro:arg name="namespace" default=""/>
+    <xacro:arg name="description_calibration_dir" default="$(find tiago_description_calibration)/urdf/calibration"/>
+    <xacro:arg name="extrinsic_calibration_dir" default="$(find tiago_description_calibration)/urdf/calibration"/>
     <xacro:property name="end_effector" value="$(arg end_effector)" />
     <xacro:property name="ft_sensor" value="$(arg ft_sensor)" />
@@ -23,4 +25,6 @@
     <xacro:property name="is_multiple" value="$(arg multiple)" />
     <xacro:property name="nsp" value="$(arg namespace)" />
+ <xacro:property name="description_calibration_dir"       value="${arg description_calibration_dir}"/>
+  <xacro:property name="extrinsic_calibration_dir"       value="${arg extrinsic_calibration_dir}"/>
   <xacro:if value="${end_effector not in ['false', 'pal-gripper', 'pal-hey5', 'schunk-wsg']}">
     <xacro:wrong_end_effector/>
