Commit message: Some updates

File: robots/tiago_steel_without_wheels.urdf (robot description, URDF)
Before this commit: robot tiago, 55 links, 54 joints
Joints:
- removed joint gripper_grasping_frame_joint
- added joint gripper__joint: type fixed, parent gripper_link, child gripper_grasping_frame, origin xyz=0 0 -0.12 rpy=-1.5708 1.5708 0
